File: pcb-test.kicad_pcb (KiCad board)
At the start: 2 copper layers, 33 parts, among them U1 ProMicro

Commit message: Finished PCB design
Parts:
- moved D16 131.4 mm to (201.6, 146.8), turned to 90 degrees
- moved D12 125.5 mm to (182.6, 146.8), turned to 90 degrees
- moved D8 122.5 mm to (163.5, 146.8), turned to 90 degrees
- moved D11 119.3 mm to (182.6, 127.8), turned to 90 degrees
- moved D4 117.2 mm to (144.5, 146.8), turned to 90 degrees
- moved D15 113.0 mm to (201.6, 127.8), turned to 90 degrees
- moved D7 112.5 mm to (163.5, 127.8), turned to 90 degrees
- moved D10 111.3 mm to (182.6, 108.7), turned to 90 degrees
- moved D13 110.9 mm to (201.6, 89.7), turned to 90 degrees
- moved D14 110.8 mm to (201.6, 108.7), turned to 90 degrees
- moved D3 109.0 mm to (144.5, 127.8), turned to 90 degrees
- moved D5 105.6 mm to (163.5, 89.7), turned to 90 degrees
- moved D6 104.0 mm to (163.5, 108.7), turned to 90 degrees
- moved D2 99.6 mm to (144.5, 108.7), turned to 90 degrees
- moved U1 98.5 mm to (116.7, 92.1), turned to 270 degrees
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Routing:
- net col3: track 0.00 -> 143.6 mm
- net row3: track 0.00 -> 134.0 mm
- net col2: track 0.00 -> 119.8 mm
- net row2: track 0.00 -> 118.5 mm
- net row1: track 0.00 -> 107.2 mm
- net col1: track 0.00 -> 95.9 mm
- net row0: track 0.00 -> 95.2 mm
- net col0: track 0.00 -> 67.6 mm
- net Net-(D5-Pad2): track 0.00 -> 6.03 mm
- net Net-(D1-Pad2): track 0.00 -> 6.03 mm
- net Net-(D8-Pad2): track 0.00 -> 6.03 mm
- net Net-(D7-Pad2): track 0.00 -> 6.03 mm
- net Net-(D6-Pad2): track 0.00 -> 6.03 mm
- net Net-(D4-Pad2): track 0.00 -> 6.03 mm
- net Net-(D3-Pad2): track 0.00 -> 6.03 mm
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Other:
- board outline added: 100 x 76.2 mm

Commit message: Small adjustments
Other:
- board size 100 x 76.2 mm -> 103.2 x 82.5 mm
Changed lines of the file:
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@@
   (general
     (thickness 1.6)
-    (drawings 8)
-    (tracks 122)
+    (drawings 18)
+    (tracks 123)
     (zones 0)
     (modules 33)
@@
     (37 F.SilkS user)
     (38 B.Mask user)
-    (39 F.Mask user)
+    (39 F.Mask user hide)
     (40 Dwgs.User user)
     (41 Cmts.User user)
@@
     (solder_mask_min_width 0.25)
     (aux_axis_origin 0 0)
-    (visible_elements FFFFE77F)
+    (visible_elements FFFFF77F)
     (pcbplotparams
       (layerselection 0x010fc_ffffffff)
-      (usegerberextensions false)
+      (usegerberextensions true)
       (usegerberattributes false)
       (usegerberadvancedattributes false)
@@
       (viasonmask false)
       (mode 1)
-      (useauxorigin false)
+      (useauxorigin true)
       (hpglpennumber 1)
       (hpglpenspeed 20)
@@
       (plotinvisibletext false)
       (padsonsilk false)
-      (subtractmaskfromsilk false)
+      (subtractmaskfromsilk true)
       (outputformat 1)
       (mirror false)
-      (drillshape 1)
+      (drillshape 0)
       (scaleselection 1)
-      (outputdirectory ""))
+      (outputdirectory "gerbers/"))
   )
   (net 0 "")
@@
     )
   )
-  (gr_line (start 200.81875 152.4) (end 105.56875 152.4) (layer Edge.Cuts) (width 0.05))
-  (gr_line (start 203.2 78.58125) (end 203.2 150.01875) (layer Edge.Cuts) (width 0.05))
-  (gr_line (start 105.56875 76.2) (end 200.81875 76.2) (layer Edge.Cuts) (width 0.05))
+  (gr_circle (center 203.2 76.2) (end 203.2 73.81875) (layer Edge.Cuts) (width 0.05))
+  (gr_circle (center 203.2 152.4) (end 203.2 154.78125) (layer Edge.Cuts) (width 0.05))
+  (gr_circle (center 106.3625 152.4) (end 106.3625 154.78125) (layer Edge.Cuts) (width 0.05))
+  (gr_circle (center 106.3625 76.2) (end 104.775 74.6125) (layer Edge.Cuts) (width 0.05))
+  (gr_line (start 203.99375 155.575) (end 200.81875 155.575) (layer Edge.Cuts) (width 0.05))
+  (gr_line (start 206.375 153.19375) (end 206.375 150.01875) (layer Edge.Cuts) (width 0.05))
+  (gr_line (start 203.99375 73.025) (end 200.81875 73.025) (layer Edge.Cuts) (width 0.05))
+  (gr_line (start 206.375 75.40625) (end 206.375 78.58125) (layer Edge.Cuts) (width 0.05))
+  (gr_line (start 103.1875 78.58125) (end 103.1875 75.40625) (layer Edge.Cuts) (width 0.05))
+  (gr_line (start 103.1875 150.01875) (end 103.1875 153.19375) (layer Edge.Cuts) (width 0.05))
+  (gr_line (start 200.81875 155.575) (end 105.56875 155.575) (layer Edge.Cuts) (width 0.05))
+  (gr_line (start 206.375 78.58125) (end 206.375 150.01875) (layer Edge.Cuts) (width 0.05))
+  (gr_line (start 105.56875 73.025) (end 200.81875 73.025) (layer Edge.Cuts) (width 0.05))
   (gr_line (start 103.1875 150.01875) (end 103.1875 78.58125) (layer Edge.Cuts) (width 0.05))
-  (gr_arc (start 105.56875 150.01875) (end 103.1875 150.01875) (angle -90) (layer Edge.Cuts) (width 0.05))
-  (gr_arc (start 105.56875 78.58125) (end 105.56875 76.2) (angle -90) (layer Edge.Cuts) (width 0.05))
-  (gr_arc (start 200.81875 150.01875) (end 200.81875 152.4) (angle -90) (layer Edge.Cuts) (width 0.05))
-  (gr_arc (start 200.81875 78.58125) (end 203.2 78.58125) (angle -90) (layer Edge.Cuts) (width 0.05))
+  (gr_arc (start 105.56875 153.19375) (end 103.1875 153.19375) (angle -90) (layer Edge.Cuts) (width 0.05))
+  (gr_arc (start 105.56875 75.40625) (end 105.56875 73.025) (angle -90) (layer Edge.Cuts) (width 0.05))
+  (gr_arc (start 203.99375 153.19375) (end 203.99375 155.575) (angle -90) (layer Edge.Cuts) (width 0.05))
+  (gr_arc (start 203.99375 75.40625) (end 206.375 75.40625) (angle -90) (layer Edge.Cuts) (width 0.05))
   (segment (start 143.002 80.61325) (end 144.4625 82.07375) (width 0.25) (layer B.Cu) (net 1))
   (segment (start 139.03325 80.61325) (end 143.002 80.61325) (width 0.25) (layer B.Cu) (net 1))
@@
   (segment (start 143.002 137.76325) (end 144.4625 139.22375) (width 0.25) (layer B.Cu) (net 7))
   (segment (start 139.03325 137.76325) (end 143.002 137.76325) (width 0.25) (layer B.Cu) (net 7))
-  (segment (start 201.6125 146.84375) (end 201.6125 150.8125) (width 0.25) (layer B.Cu) (net 8))
-  (segment (start 201.6125 150.8125) (end 182.5625 150.8125) (width 0.25) (layer B.Cu) (net 8))
   (segment (start 182.5625 146.84375) (end 182.5625 150.8125) (width 0.25) (layer B.Cu) (net 8))
   (segment (start 182.5625 150.8125) (end 163.5125 150.8125) (width 0.25) (layer B.Cu) (net 8))
@@
   (segment (start 124.30125 106.045) (end 126.52375 106.045) (width 0.25) (layer B.Cu) (net 8))
   (segment (start 126.52375 106.045) (end 126.52375 140.0175) (width 0.25) (layer B.Cu) (net 8))
+  (segment (start 201.6125 146.84375) (end 201.6125 150.01875) (width 0.25) (layer B.Cu) (net 8))
+  (segment (start 201.6125 150.01875) (end 200.81875 150.8125) (width 0.25) (layer B.Cu) (net 8))
+  (segment (start 200.81875 150.8125) (end 182.5625 150.8125) (width 0.25) (layer B.Cu) (net 8))
   (segment (start 162.052 80.61325) (end 163.5125 82.07375) (width 0.25) (layer B.Cu) (net 9))
   (segment (start 158.08325 80.61325) (end 162.052 80.61325) (width 0.25) (layer B.Cu) (net 9))
